Commit message: 4

File: agv_description/urdf/agv_for_line_following.urdf.xacro (robot description, xacro)
@@ -7,9 +7,9 @@
     <parent link="base_footprint"/>
     <child link="base_link"/>
-    <origin xyz="0.0 0.0 0.1" rpy="0 0 1.57"/>
+    <origin xyz="0.0 0.0 0.12" rpy="0 0 0"/>
   </joint>
   <link name="base_link">
     <visual>
-      <origin xyz="0.0 0 0.12" rpy="0 0 1.57"/>
+      <origin xyz="0.0 0 0.07" rpy="0 0 1.57"/>
       <geometry>
         <mesh filename="package://agv_description/meshes/bases/agv_base.stl" scale="0.001 0.001 0.001"/>
@@ -34,5 +34,5 @@
     <parent link="base_link"/>
     <child link="wheel_left_link"/>
-    <origin xyz="-0.4 0.0 0.075" rpy="1.57 0 0"/>
+    <origin xyz="-0.4 0.0 0.075" rpy="-1.57 0 0"/>
     <axis xyz="0 0 1"/>
   </joint>
@@ -45,10 +45,10 @@
       <material name="white"/>
     </visual-->
-    <collision>
+    <!--collision>
       <origin xyz="0.0 0 0" rpy="0 0 0"/>
       <geometry>
         <cylinder length="0.22" radius="0.09"/>
       </geometry>
-    </collision>
+    </collision-->
     <inertial>
       <origin xyz="0 0 0" />
@@ -73,10 +73,10 @@
       <material name="dark"/>
     </visual-->
-    <collision>
+    <!--collision>
       <origin xyz="0 0 0" rpy="0 0 0"/>
       <geometry>
         <cylinder length="0.22" radius="0.09"/>
       </geometry>
-    </collision>
+    </collision-->
     <inertial>
       <origin xyz="0 0 0" />
