Commit message: 3

File: agv_description/urdf/agv_for_line_following.gazebo.xacro (robot description, xacro)
@@ -43,5 +43,5 @@
   </gazebo>
   <gazebo>
-    <plugin name="turtlebot3_burger_controller" filename="libgazebo_ros_diff_drive.so">
+    <plugin name="agv_controller" filename="libgazebo_ros_diff_drive.so">
       <commandTopic>cmd_vel</commandTopic>
       <odometryTopic>odom</odometryTopic>

File: agv_description/urdf/agv_for_line_following.urdf.xacro (robot description, xacro)
@@ -7,9 +7,9 @@
     <parent link="base_footprint"/>
     <child link="base_link"/>
-    <origin xyz="0.0 0.0 0.05" rpy="0 0 1.57"/>
+    <origin xyz="0.0 0.0 0.1" rpy="0 0 1.57"/>
   </joint>
   <link name="base_link">
     <visual>
-      <origin xyz="0.0 0 0.05" rpy="0 0 1.57"/>
+      <origin xyz="0.0 0 0.12" rpy="0 0 1.57"/>
       <geometry>
         <mesh filename="package://agv_description/meshes/bases/agv_base.stl" scale="0.001 0.001 0.001"/>
@@ -18,5 +18,5 @@
     </visual>
     <collision>
-      <origin xyz="0.0 0 0.05" rpy="0 0 1.57"/>
+      <origin xyz="0.0 0 0.12" rpy="0 0 0"/>
       <geometry>
         <box size="1.0 0.8 0.24"/>
@@ -25,8 +25,8 @@
     <inertial>
       <origin xyz="0 0 0" rpy="0 0 0"/>
-      <mass value="100"/>
-      <inertia ixx="0" ixy="0" ixz="0"
-               iyy="0" iyz="0"
-               izz="0" />
+      <mass value="10"/>
+      <inertia ixx="6.48224043" ixy="5.06925791e-2" ixz="2.42332909e-2"
+               iyy="2.65332346" iyz="-1.25236226e-2"
+               izz="7.7704931" />
     </inertial>
   </link>
@@ -34,5 +34,5 @@
     <parent link="base_link"/>
     <child link="wheel_left_link"/>
-    <origin xyz="0.0 -0.35 0.18" rpy="0 0 0"/>
+    <origin xyz="-0.4 0.0 0.075" rpy="1.57 0 0"/>
     <axis xyz="0 0 1"/>
   </joint>
@@ -45,16 +45,16 @@
       <material name="white"/>
     </visual-->
-    <!--collision>
-      <origin xyz="0.0 -0.35 0.18" rpy="0 0 0"/>
+    <collision>
+      <origin xyz="0.0 0 0" rpy="0 0 0"/>
       <geometry>
-        <cylinder length="0.22" radius="0.18"/>
+        <cylinder length="0.22" radius="0.09"/>
       </geometry>
-    </collision-->
+    </collision>
     <inertial>
       <origin xyz="0 0 0" />
-      <mass value="15.0" />
-      <inertia ixx="0" ixy="0" ixz="0"
-               iyy="0" iyz="0"
-               izz="0" />
+      <mass value="1.5" />
+      <inertia ixx="4.05139588e-2" ixy="5.22245694e-3" ixz="1.40418470e-3"
+               iyy="4.88302387e-2" iyz="1.86962703e-3"
+               izz="4.58877115e-2" />
       </inertial>
   </link>
@@ -62,5 +62,5 @@
     <parent link="base_link"/>
     <child link="wheel_right_link"/>
-    <origin xyz="0.0 0.28 0.16" rpy="0 0 0"/>
+    <origin xyz="0.3 0.0 0.075" rpy="-1.57 0 0"/>
     <axis xyz="0 0 1"/>
   </joint>
@@ -73,16 +73,16 @@
       <material name="dark"/>
     </visual-->
-    <!--collision>
-      <origin xyz="0.0 0.28 0.16" rpy="0 0 0"/>
+    <collision>
+      <origin xyz="0 0 0" rpy="0 0 0"/>
       <geometry>
-        <cylinder length="0.22" radius="0.18"/>
+        <cylinder length="0.22" radius="0.09"/>
       </geometry>
-    </collision-->
+    </collision>
     <inertial>
       <origin xyz="0 0 0" />
-      <mass value="15.0" />
-      <inertia ixx="0" ixy="0" ixz="0"
-               iyy="0" iyz="0"
-               izz="0" />
+      <mass value="1.5" />
+      <inertia ixx="4.05139588e-2" ixy="5.22245694e-3" ixz="1.40418470e-3"
+               iyy="4.88302387e-2" iyz="1.86962703e-3"
+               izz="4.58877115e-2" />
       </inertial>
   </link>
@@ -101,9 +101,9 @@
     <inertial>
       <origin xyz="0 0 0" />
-      <mass value="5.0" />
-      <inertia ixx="0.00" ixy="0.0" ixz="0.0"
-               iyy="0.00" iyz="0.0"
-               izz="0.00" />
-    </inertial>
+      <mass value="0.5" />
+      <inertia ixx="3.21479325e-03" ixy="-1.62611171e-05" ixz="-7.91864042e-04"
+               iyy="4.53599232e-03" iyz="-3.15202900e-05"
+               izz="2.24290037e-03" />
+      </inertial>
   </link>
   <joint name="caster_right_joint" type="fixed">
@@ -121,9 +121,9 @@
     <inertial>
       <origin xyz="0 0 0" />
-      <mass value="5.0" />
-      <inertia ixx="0.00" ixy="0.0" ixz="0.0"
-               iyy="0.00" iyz="0.0"
-               izz="0.00" />
-    </inertial>
+      <mass value="0.5" />
+      <inertia ixx="3.21479325e-03" ixy="-1.62611171e-05" ixz="-7.91864042e-04"
+               iyy="4.53599232e-03" iyz="-3.15202900e-05"
+               izz="2.24290037e-03" />
+      </inertial>
   </link>
 </robot>

Commit message: add two wheel control and camera

File: agv_description/urdf/agv_for_line_following.gazebo.xacro (robot description, xacro)
@@ -42,24 +42,105 @@
     <material>Gazebo/FlatBlack</material>
   </gazebo>
+    <!-- camera -->
+  <gazebo reference="camera_link">
+    <sensor type="camera" name="camera1">
+      <update_rate>30.0</update_rate>
+      <camera name="head">
+        <horizontal_fov>1.3962634</horizontal_fov>
+        <image>
+          <width>800</width>
+          <height>800</height>
+          <format>R8G8B8</format>
+        </image>
+        <clip>
+          <near>0.02</near>
+          <far>300</far>
+        </clip>
+        <noise>
+          <type>gaussian</type>
+          <!-- Noise is sampled independently per pixel on each frame.
+               That pixel's noise value is added to each of its color
+               channels, which at that point lie in the range [0,1]. -->
+          <mean>0.0</mean>
+          <stddev>0.007</stddev>
+        </noise>
+      </camera>
+      <plugin name="camera_controller" filename="libgazebo_ros_camera.so">
+        <alwaysOn>true</alwaysOn>
+        <updateRate>0.0</updateRate>
+        <cameraName>agv/camera1</cameraName>
+        <imageTopicName>image_raw</imageTopicName>
+        <cameraInfoTopicName>camera_info</cameraInfoTopicName>
+        <frameName>camera_link_optical</frameName>
+        <!-- setting hackBaseline to anything but 0.0 will cause a misalignment
+            between the gazebo sensor image and the frame it is supposed to
+            be attached to -->
+        <hackBaseline>0.0</hackBaseline>
+        <distortionK1>0.0</distortionK1>
+        <distortionK2>0.0</distortionK2>
+        <distortionK3>0.0</distortionK3>
+        <distortionT1>0.0</distortionT1>
+        <distortionT2>0.0</distortionT2>
+        <CxPrime>0</CxPrime>
+        <Cx>0.0</Cx>
+        <Cy>0.0</Cy>
+        <focalLength>0.0</focalLength>
+      </plugin>
+    </sensor>
+  </gazebo>
   <gazebo>
-    <plugin name="agv_controller" filename="libgazebo_ros_diff_drive.so">
-      <commandTopic>cmd_vel</commandTopic>
+    <plugin name="tricycle_drive_controller1" filename="libgazebo_ros_tricycle_drive.so">
+      <rosDebugLevel>Debug</rosDebugLevel>
+      <robotNamespace></robotNamespace>
+      <publishWheelTF>false</publishWheelTF>
+      <publishWheelJointState>true</publishWheelJointState>
+      <alwaysOn>true</alwaysOn>
+      <steeringJoint>wheel_left_steering_joint</steeringJoint>
+      <actuatedWheelJoint>wheel_left_joint</actuatedWheelJoint>
+      <encoderWheelLeftJoint>wheel_left_joint</encoderWheelLeftJoint>
+      <encoderWheelRightJoint>wheel_right_joint</encoderWheelRightJoint>
+      <actuatedWheelDiameter>0.180</actuatedWheelDiameter>
+      <encoderWheelDiameter>0.180</encoderWheelDiameter>
+      <encoderWheelSeparation>0.7</encoderWheelSeparation>
+      <commandTopic>cmd_vel1</commandTopic>
       <odometryTopic>odom</odometryTopic>
       <odometryFrame>odom</odometryFrame>
       <odometrySource>world</odometrySource>
-      <publishOdomTF>true</publishOdomTF>
       <robotBaseFrame>base_footprint</robotBaseFrame>
+      <updateRate>10.0</updateRate>
+      <wheelAcceleration>1.8</wheelAcceleration>
+      <wheelDeceleration>5.0</wheelDeceleration>
+      <wheelSpeedTolerance>0.05</wheelSpeedTolerance>
+      <wheelTorque>20</wheelTorque>
+      <steeringSpeed>0.4</steeringSpeed>
+      <steeringAngleTolerance>0.02</steeringAngleTolerance>
+    </plugin>
+  </gazebo>
+    <gazebo>
+    <plugin name="tricycle_drive_controller2" filename="libgazebo_ros_tricycle_drive.so">
+      <rosDebugLevel>Debug</rosDebugLevel>
+      <robotNamespace></robotNamespace>
       <publishWheelTF>false</publishWheelTF>
-      <publishTf>true</publishTf>
-      <publishWheelJointState>true</publishWheelJointState>
-      <legacyMode>false</legacyMode>
-      <updateRate>30</updateRate>
-      <leftJoint>wheel_left_joint</leftJoint>
-      <rightJoint>wheel_right_joint</rightJoint>
-      <wheelSeparation>0.700</wheelSeparation>
-      <wheelDiameter>0.180</wheelDiameter>
-      <wheelAcceleration>1</wheelAcceleration>
-      <wheelTorque>10</wheelTorque>
-      <rosDebugLevel>na</rosDebugLevel>
+      <publishWheelJointState>false</publishWheelJointState>
+      <alwaysOn>true</alwaysOn>
+      <steeringJoint>wheel_right_steering_joint</steeringJoint>
+      <actuatedWheelJoint>wheel_right_joint</actuatedWheelJoint>
+      <encoderWheelLeftJoint>wheel_left_joint</encoderWheelLeftJoint>
+      <encoderWheelRightJoint>wheel_right_joint</encoderWheelRightJoint>
+      <actuatedWheelDiameter>0.180</actuatedWheelDiameter>
+      <encoderWheelDiameter>0.180</encoderWheelDiameter>
+      <encoderWheelSeparation>0.7</encoderWheelSeparation>
+      <commandTopic>cmd_vel2</commandTopic>
+      <odometryTopic>odom1</odometryTopic>
+      <odometryFrame>odom1</odometryFrame>
+      <odometrySource>world</odometrySource>
+      <robotBaseFrame>base_footprint</robotBaseFrame>
+      <updateRate>10.0</updateRate>
+      <wheelAcceleration>1.8</wheelAcceleration>
+      <wheelDeceleration>5.0</wheelDeceleration>
+      <wheelSpeedTolerance>0.05</wheelSpeedTolerance>
+      <wheelTorque>20</wheelTorque>
+      <steeringSpeed>0.4</steeringSpeed>
+      <steeringAngleTolerance>0.02</steeringAngleTolerance>
     </plugin>
   </gazebo>

File: agv_description/urdf/agv_for_line_following.urdf.xacro (robot description, xacro)
@@ -18,5 +18,5 @@
     </visual>
     <collision>
-      <origin xyz="0.0 0 0.12" rpy="0 0 0"/>
+      <origin xyz="0.0 0 0.22" rpy="0 0 0"/>
       <geometry>
         <box size="1.0 0.8 0.24"/>
@@ -31,24 +31,160 @@
     </inertial>
   </link>
+  <joint name="caster_left_joint" type="fixed">
+    <parent link="base_link"/>
+    <child link="caster_left_link"/>
+    <origin xyz="0 0.3118 0.03" rpy="0 0 1.57"/>
+  </joint>
+  <link name="caster_left_link">
+    <!--collision>
+      <origin xyz="0 0 0" rpy="0 0 0"/>
+       <geometry>
+        <mesh filename="package://agv_description/meshes/wheels/caster_left.stl" scale="0.001 0.001 0.001"/>
+      </geometry>
+    </collision-->
+    <inertial>
+      <origin xyz="0 0 0" />
+      <mass value="0.5" />
+      <inertia ixx="3.21479325e-03" ixy="-1.62611171e-05" ixz="-7.91864042e-04"
+               iyy="4.53599232e-03" iyz="-3.15202900e-05"
+               izz="2.24290037e-03" />
+      </inertial>
+  </link>
+  <joint name="caster_right_joint" type="fixed">
+    <parent link="base_link"/>
+    <child link="caster_right_link"/>
+    <origin xyz="0 -0.3118 0.03" rpy="0 0 1.57"/>
+  </joint>
+  <link name="caster_right_link">
+    <!--collision>
+      <origin xyz="0 0 0" rpy="0 0 0"/>
+      <geometry>
+        <mesh filename="package://agv_description/meshes/wheels/caster_right.stl" scale="0.001 0.001 0.001"/>
+      </geometry>
+    </collision-->
+    <inertial>
+      <origin xyz="0 0 0" />
+      <mass value="0.5" />
+      <inertia ixx="3.21479325e-03" ixy="-1.62611171e-05" ixz="-7.91864042e-04"
+               iyy="4.53599232e-03" iyz="-3.15202900e-05"
+               izz="2.24290037e-03" />
+      </inertial>
+  </link>
+  <joint name="camera_joint" type="fixed">
+    <axis xyz="0 1 0" />
+    <origin xyz="0.46 0.03 0" rpy="0 0 0"/>
+    <parent link="base_link"/>
+    <child link="camera_link"/>
+  </joint>
+  <!-- Camera -->
+  <link name="camera_link">
+    <collision>
+      <origin xyz="0 0 0" rpy="0 0 0"/>
+      <geometry>
+	      <box size="0.01 0.01 0.01"/>
+      </geometry>
+    </collision>
+    <visual>
+      <origin xyz="0 0 0" rpy="0 0 0"/>
+      <geometry>
+	        <box size="0.01 0.01 0.01"/>
+      </geometry>
+      <material name="red"/>
+    </visual>
+    <inertial>
+      <mass value="1e-5" />
+      <origin xyz="0 0 0" rpy="0 0 0"/>
+      <inertia ixx="1e-6" ixy="0" ixz="0" iyy="1e-6" iyz="0" izz="1e-6" />
+    </inertial>
+  </link>
+  <!-- generate an optical frame http://www.ros.org/reps/rep-0103.html#suffix-frames
+      so that ros and opencv can operate on the camera frame correctly -->
+  <joint name="camera_optical_joint" type="fixed">
+    <!-- these values have to be these values otherwise the gazebo camera image
+        won't be aligned properly with the frame it is supposedly originating from -->
+    <origin xyz="0 0 0" rpy="-1.57 0 -1.57"/>
+    <parent link="camera_link"/>
+    <child link="camera_link_optical"/>
+  </joint>
+  <link name="camera_link_optical">
+  </link>
+    <!-- steering joint -->
+  <joint name="wheel_left_steering_joint" type="continuous">
+    <origin xyz="-0.4 0.0 0.075" rpy="0 0 0"/>
+    <parent link="base_link"/>
+    <child link="wheel_left_steering"/>
+    <axis xyz="0 0 1"/>
+    <anchor xyz="0 0 0"/>
+    <limit effort="100" velocity="100" k_velocity="0"/>
+    <joint_properties damping="0.0" friction="0.0"/>
+  </joint>
+  <link name="wheel_left_steering">
+    <visual name="wheel_left_steering_visual">
+      <origin xyz="0 0 0" rpy="0 0 0"/>
+      <geometry name="wheel_left_steering_geometry">
+        <cylinder radius="0.01" length="0.05"/>
+      </geometry>
+      <material name="blue"/>
+    </visual>
+    <inertial>
+      <origin xyz="0 0 0" />
+      <mass value="0.001" />
+      <inertia ixx="3.21479325e-09" ixy="1.62611171e-9" ixz="7.91864042e-9"
+               iyy="4.53599232e-09" iyz="3.15202900e-9"
+               izz="2.24290037e-09" />
+      </inertial>
+  </link>
+  <gazebo reference="wheel_left_steering">
+    <material value="Gazebo/Blue"/>
+  </gazebo>
+  <!-- steering joint -->
+  <joint name="wheel_right_steering_joint" type="continuous">
+    <origin xyz="0.3 0.0 0.075" rpy="0 0 0"/>
+    <parent link="base_link"/>
+    <child link="wheel_right_steering"/>
+    <axis xyz="0 0 1"/>
+    <anchor xyz="0 0 0"/>
+    <limit effort="100" velocity="100" k_velocity="0"/>
+    <joint_properties damping="0.0" friction="0.0"/>
+  </joint>
+  <link name="wheel_right_steering">
+    <visual name="wheel_right_steering_visual">
+      <origin xyz="0 0 0" rpy="0 0 0"/>
+      <geometry name="wheel_right_steering_geometry">
+        <cylinder radius="0.01" length="0.05"/>
+      </geometry>
+      <material name="blue"/>
+    </visual>
+    <inertial>
+      <origin xyz="0 0 0" />
+      <mass value="0.001" />
+      <inertia ixx="3.21479325e-09" ixy="1.62611171e-9" ixz="7.91864042e-9"
+               iyy="4.53599232e-09" iyz="3.15202900e-9"
+               izz="2.24290037e-09" />
+      </inertial>
+  </link>
+  <gazebo reference="wheel_right_steering">
+    <material value="Gazebo/Blue"/>
+  </gazebo>
   <joint name="wheel_left_joint" type="continuous">
-    <parent link="base_link"/>
+    <parent link="wheel_left_steering"/>
     <child link="wheel_left_link"/>
-    <origin xyz="-0.4 0.0 0.075" rpy="-1.57 0 0"/>
+    <origin xyz="0 0 0" rpy="-1.57 0 0"/>
     <axis xyz="0 0 1"/>
   </joint>
   <link name="wheel_left_link">
-    <!--visual>
-      <origin xyz="0.0 -0.35 0.18" rpy="0 0 0"/>
-      <geometry>
-        <mesh filename="package://agv_description/meshes/wheels/wheel_left.stl" scale="0.001 0.001 0.001"/>
-      </geometry>
-      <material name="white"/>
-    </visual-->
-    <!--collision>
+    <visual>
       <origin xyz="0.0 0 0" rpy="0 0 0"/>
       <geometry>
         <cylinder length="0.22" radius="0.09"/>
       </geometry>
-    </collision-->
+      <material name="red"/>
+    </visual>
+    <collision>
+      <origin xyz="0.0 0 0" rpy="0 0 0"/>
+      <geometry>
+        <cylinder length="0.22" radius="0.09"/>
+      </geometry>
+    </collision>
     <inertial>
       <origin xyz="0 0 0" />
@@ -60,23 +196,23 @@
   </link>
   <joint name="wheel_right_joint" type="continuous">
-    <parent link="base_link"/>
+    <parent link="wheel_right_steering"/>
     <child link="wheel_right_link"/>
-    <origin xyz="0.3 0.0 0.075" rpy="-1.57 0 0"/>
+    <origin xyz="0 0.0 0" rpy="-1.57 0 0"/>
     <axis xyz="0 0 1"/>
   </joint>
   <link name="wheel_right_link">
-    <!--visual>
-      <origin xyz="0.0 0.28 0.16" rpy="0 0 3.14"/>
-      <geometry>
-        <mesh filename="package://agv_description/meshes/wheels/wheel_right.stl" scale="0.001 0.001 0.001"/>
-      </geometry>
-      <material name="dark"/>
-    </visual-->
-    <!--collision>
-      <origin xyz="0 0 0" rpy="0 0 0"/>
-      <geometry>
-        <cylinder length="0.22" radius="0.09"/>
-      </geometry>
-    </collision-->
+    <visual>
+      <origin xyz="0.0 0 0" rpy="0 0 0"/>
+      <geometry>
+        <cylinder length="0.22" radius="0.09"/>
+      </geometry>
+      <material name="red"/>
+    </visual>
+    <collision>
+      <origin xyz="0 0 0" rpy="0 0 0"/>
+      <geometry>
+        <cylinder length="0.22" radius="0.09"/>
+      </geometry>
+    </collision>
     <inertial>
       <origin xyz="0 0 0" />
@@ -87,43 +223,3 @@
       </inertial>
   </link>
-  <joint name="caster_left_joint" type="fixed">
-    <parent link="base_link"/>
-    <child link="caster_left_link"/>
-    <origin xyz="0 0.3118 0.03" rpy="0 0 1.57"/>
-  </joint>
-  <link name="caster_left_link">
-    <!--collision>
-      <origin xyz="0 0 0" rpy="0 0 0"/>
-       <geometry>
-        <mesh filename="package://agv_description/meshes/wheels/caster_left.stl" scale="0.001 0.001 0.001"/>
-      </geometry>
-    </collision-->
-    <inertial>
-      <origin xyz="0 0 0" />
-      <mass value="0.5" />
-      <inertia ixx="3.21479325e-03" ixy="-1.62611171e-05" ixz="-7.91864042e-04"
-               iyy="4.53599232e-03" iyz="-3.15202900e-05"
-               izz="2.24290037e-03" />
-      </inertial>
-  </link>
-  <joint name="caster_right_joint" type="fixed">
-    <parent link="base_link"/>
-    <child link="caster_right_link"/>
-    <origin xyz="0 -0.3118 0.03" rpy="0 0 1.57"/>
-  </joint>
-  <link name="caster_right_link">
-    <!--collision>
-      <origin xyz="0 0 0" rpy="0 0 0"/>
-      <geometry>
-        <mesh filename="package://agv_description/meshes/wheels/caster_right.stl" scale="0.001 0.001 0.001"/>
-      </geometry>
-    </collision-->
-    <inertial>
-      <origin xyz="0 0 0" />
-      <mass value="0.5" />
-      <inertia ixx="3.21479325e-03" ixy="-1.62611171e-05" ixz="-7.91864042e-04"
-               iyy="4.53599232e-03" iyz="-3.15202900e-05"
-               izz="2.24290037e-03" />
-      </inertial>
-  </link>
 </robot>
